File: KiCad/VectorDock_RevA/usb_hub.kicad_sch (KiCad schematic)
At the start: 23 parts, among them U1 USB5744_2G, Y1 ABM8G-25.000MHZ-B4Y-T

Commit message: Worked on hub sheet
Parts:
- added C15, C16: 100 nF, symbol Device:C_Small
- added C20, C21: 330 nF, symbol Device:C_Small
- added J1: HOST_USB_C_CAPTIVE, symbol Connector_Generic:Conn_01x10
- added U2: TPD4E05U06DQAR, DQA0010A, symbol VectorDock:TPD4E05U06DQAR
- added U3: TPD2EUSB30ADRTR, DRT3, symbol VectorDock:TPD2EUSB30ADRTR
Connections:
- net GND: now also J1.9 (Pin_9), U2.3 (GND), U2.8 (GND), U3.3 (GND)
- net UP_USB2_DP: now reaches U1.45 (USB2UP_DP)
- net UP_USB2_DP: now also J1.5 (Pin_5), U3.1 (D+)
- net UP_USB2_DM: now reaches U1.46 (USB2UP_DM)
- net UP_USB2_DM: now also J1.6 (Pin_6), U3.2 (D-)
- net at U1.47 (USB3UP_TXDP): now also C15.1
- net at U1.48 (USB3UP_TXDM): now also C16.1
- net at U1.50 (USB3UP_RXDP): now also C21.1
- net at U1.51 (USB3UP_RXDM): now also C20.1
- new net HOST_CC: J1.7 (Pin_7)
- new net HOST_VBUS: J1.8 (Pin_8)
- new net SHIELD: J1.10 (Pin_10)
- new net UP_SS_RX_N: C20.2, J1.4 (Pin_4), U2.5 (D2-)
- new net UP_SS_RX_P: C21.2, J1.3 (Pin_3), U2.4 (D2+)
- new net UP_SS_TX_N: C16.2, J1.2 (Pin_2), U2.2 (D1-)
- new net UP_SS_TX_P: C15.2, J1.1 (Pin_1), U2.1 (D1+)
Other:
- moved on the sheet: C1, C10, C11, C12, C13, C14, C17, C18, C19, C2, C3, C4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

Commit message: Worked on USB PC
Connections:
- net XTALI: now reaches C17.1, U1.54 (XTALI/CLK_IN), Y1.1
- net XTALO: now reaches C18.1, U1.53 (XTALO), Y1.3
Other:
- moved on the sheet: C17, C18, U3, Y1
