File: KiCad/VectorDock_RevA/usb_pd.kicad_sch (KiCad schematic)
At the start: 0 parts

Commit message: Worked on hub sheet
Parts:
- added IC1: TPS25752ASRSMR, QFN40P400X400X100-33N-D, symbol VectorDock:TPS25752ASRSMR
- added IC2: TPS25751DREFR, TPS25730ADREFR, symbol VectorDock:TPS25751DREFR
- added U4: TPS55288RPMR, TPS55288RPMR:IC_TPS55288RPMR, symbol VectorDock:TPS55288RPMR
Connections:
- new net: U4.11 (VOUT), U4.26 (VOUT)
- new net: U4.21 (SW2), U4.25 (SW2)
- new net PGND: U4.24 (PGND), U4.9 (PGND)

Commit message: Worked on USB PC
Parts:
- added C22, C23, C24: 10 µF, symbol Device:C_Small
- added C25: 4.7 µF, 25 V, symbol Device:C_Small
- added C26, C27: 330 pF, symbol Device:C_Small
- added C28, C29: 22 µF, symbol Device:C_Small
- added C30: 100 nF, symbol Device:C_Small
- added J2: USB_C_Receptacle_PowerOnly_6P, symbol Connector:USB_C_Receptacle_PowerOnly_6P
- IC2: value TPS25751DREFR -> TPS25751ADREFR
Connections:
- net at IC2.1 (LDO_3V3): now also C22.1
- net GND: now reaches IC2.11 (GND_1)
- net GND: now also IC2.12 (GND_2), IC2.14 (GND_3), IC2.31 (GND_4), IC2.39 (GND_5), C22.2, C23.2, C24.1, C25.2, C26.1, C27.1, C28.1, C29.1, C30.1, J2.A12 (GND), J2.B12 (GND)
- net DRAIN: now reaches IC2.15 (DRAIN_1)
- net DRAIN: now also IC2.30 (DRAIN_2), IC2.40 (DRAIN_3)
- net PD_INPUT_BUS: now reaches IC2.20 (PPHV)
- net PD_INPUT_BUS: now also C28.2, C29.2, C30.2
- net CHG_VBUS: now reaches IC2.23 (VBUS_IN)
- net CHG_VBUS: now also IC2.32 (VBUS), C25.1, J2.A9 (VBUS), J2.B9 (VBUS)
- net CHG_CC1: now reaches IC2.28 (CC1)
- net CHG_CC1: now also C26.2, J2.A5 (CC1)
- net CHG_CC2: now reaches IC2.29 (CC2)
- net CHG_CC2: now also C27.2, J2.B5 (CC2)
- net +3V3_DOCK: now reaches IC2.38 (VIN_3V3)
- net +3V3_DOCK: now also C24.2
- net at IC2.4 (LDO_1V5): now also C23.1
- new net CHG_SHIELD: J2.SH (SHIELD)
Other:
- moved on the sheet: IC1, U4
